Commit message: Better Robot Model and Launch File

File: urdf/robot.urdf.xacro (robot description, xacro)
@@ -31,5 +31,5 @@
   <link name="left_wheel_link">
     <visual>
-      <origin xyz="0 0 0" rpy="1.5708 0 0"/>
+      <origin xyz="-.15 0 0" rpy="1.5708 0 0"/>
       <geometry>
         <cylinder radius="${wheel_radius}" length="${wheel_width}"/>
@@ -38,5 +38,5 @@
     </visual>
     <collision>
-      <origin xyz="0 0 0" rpy="1.5708 0 0"/>
+      <origin xyz="-.15 0 0" rpy="1.5708 0 0"/>
       <geometry>
         <cylinder radius="${wheel_radius}" length="${wheel_width}"/>
@@ -47,5 +47,5 @@
   <link name="right_wheel_link">
     <visual>
-      <origin xyz="0 0 0" rpy="1.5708 0 0"/>
+      <origin xyz="-.15 0 0" rpy="1.5708 0 0"/>
       <geometry>
         <cylinder radius="${wheel_radius}" length="${wheel_width}"/>
@@ -54,5 +54,5 @@
     </visual>
     <collision>
-      <origin xyz="0 0 0" rpy="1.5708 0 0"/>
+      <origin xyz="-.15 0 0" rpy="1.5708 0 0"/>
       <geometry>
         <cylinder radius="${wheel_radius}" length="${wheel_width}"/>
@@ -64,5 +64,5 @@
     <parent link="base_link"/>
     <child link="left_wheel_link"/>
-    <origin xyz="0 ${wheel_separation/2} 0"/>
+    <origin xyz="0 ${wheel_separation * 0.5 + wheel_width*0.5} -${wheel_radius * 0.5}"/>
     <axis xyz="0 1 0"/>
   </joint>
@@ -70,5 +70,5 @@
     <parent link="base_link"/>
     <child link="right_wheel_link"/>
-    <origin xyz="0 -${wheel_separation/2} 0"/>
+    <origin xyz="0 -${wheel_separation * 0.5 + wheel_width*0.5} -${wheel_radius * 0.5}"/>
     <axis xyz="0 1 0"/>
   </joint>

Commit message: Fixed Wheel Links and Gazebo World With Floor

File: urdf/robot.urdf.xacro (robot description, xacro)
@@ -31,5 +31,5 @@
   <link name="left_wheel_link">
     <visual>
-      <origin xyz="-.15 0 0" rpy="1.5708 0 0"/>
+      <origin xyz="0 0 0" rpy="1.5708 0 0"/>
       <geometry>
         <cylinder radius="${wheel_radius}" length="${wheel_width}"/>
@@ -38,14 +38,21 @@
     </visual>
     <collision>
-      <origin xyz="-.15 0 0" rpy="1.5708 0 0"/>
+      <origin xyz="0 0 0" rpy="1.5708 0 0"/>
       <geometry>
         <cylinder radius="${wheel_radius}" length="${wheel_width}"/>
       </geometry>
     </collision>
+    <inertial>
+      <mass value="0.3"/>
+      <origin xyz="0 0 0" rpy="0 0 0"/>
+      <!-- conservative inertia guess; we can refine later -->
+      <inertia ixx="0.0005" iyy="0.0005" izz="0.0005"
+              ixy="0.0" ixz="0.0" iyz="0.0"/>
+    </inertial>
   </link>
   <!-- Right Wheel -->
   <link name="right_wheel_link">
     <visual>
-      <origin xyz="-.15 0 0" rpy="1.5708 0 0"/>
+      <origin xyz="0 0 0" rpy="1.5708 0 0"/>
       <geometry>
         <cylinder radius="${wheel_radius}" length="${wheel_width}"/>
@@ -54,9 +61,16 @@
     </visual>
     <collision>
-      <origin xyz="-.15 0 0" rpy="1.5708 0 0"/>
+      <origin xyz="0 0 0" rpy="1.5708 0 0"/>
       <geometry>
         <cylinder radius="${wheel_radius}" length="${wheel_width}"/>
       </geometry>
     </collision>
+    <inertial>
+      <mass value="0.3"/>
+      <origin xyz="0 0 0" rpy="0 0 0"/>
+      <!-- conservative inertia guess; we can refine later -->
+      <inertia ixx="0.0005" iyy="0.0005" izz="0.0005"
+              ixy="0.0" ixz="0.0" iyz="0.0"/>
+    </inertial>
   </link>
   <!-- Joints -->
@@ -73,3 +87,14 @@
     <axis xyz="0 1 0"/>
   </joint>
+  <!-- Gazebo Harmonic: Thin actuator I/O for wheel joints -->
+  <gazebo>
+    <plugin filename="gz-sim-joint-controller-system"
+            name="gz::sim::systems::JointController">
+      <joint_name>left_wheel_joint</joint_name>
+    </plugin>
+    <plugin filename="gz-sim-joint-controller-system"
+            name="gz::sim::systems::JointController">
+      <joint_name>right_wheel_joint</joint_name>
+    </plugin>
+  </gazebo>
 </robot>

Commit message: Added Caster Wheel. Turning is not smooth

File: urdf/robot.urdf.xacro (robot description, xacro)
@@ -1,34 +1,78 @@
 <?xml version="1.0"?>
 <robot xmlns:xacro="http://www.ros.org/wiki/xacro" name="modular_bot">
-  <!-- Parameters -->
-  <xacro:property name="wheel_radius" value="0.05"/>
-  <xacro:property name="wheel_width" value="0.02"/>
-  <xacro:property name="wheel_separation" value="0.30"/>
-  <!-- Yellow "material" -->
-    <material name="yellow">
+  <!-- =========================
+       Parameters
+       ========================= -->
+  <!-- Base -->
+  <xacro:property name="base_length" value="0.40"/>
+  <xacro:property name="base_width"  value="0.30"/>
+  <xacro:property name="base_height" value="0.10"/>
+  <xacro:property name="base_mass"   value="5.0"/>
+  <!-- Ground clearance:
+       Positive means wheels/caster sit slightly LOWER than the base bottom,
+       so they contact ground before the body. -->
+  <xacro:property name="wheel_ground_clearance" value="0.05"/> <!-- 5 cm -->
+  <xacro:property name="caster_ground_clearance" value="0.03"/> <!-- 3 cm -->
+  <!-- Drive wheels -->
+  <xacro:property name="wheel_radius"     value="0.05"/>
+  <xacro:property name="wheel_width"      value="0.02"/>
+  <xacro:property name="wheel_separation" value="0.30"/>  <!-- center-to-center across Y -->
+  <xacro:property name="drive_wheel_x"    value="0.10"/>  <!-- shift axle forward (X) -->
+  <xacro:property name="wheel_mass"       value="0.30"/>
+  <!-- Caster (passive sphere) -->
+  <xacro:property name="caster_radius" value="0.05"/>
+  <xacro:property name="caster_x"      value="-0.15"/>
+  <xacro:property name="caster_mass"   value="0.20"/>
+  <!-- Derived Z offsets (relative to base_link centered in the box) -->
+  <!-- base bottom is at z = -base_height/2 -->
+  <!-- wheel center z: base bottom - clearance + wheel_radius -->
+  <xacro:property name="drive_wheel_z"
+                  value="${-base_height*0.5 - wheel_ground_clearance + wheel_radius}"/>
+  <!-- caster center z: base bottom - clearance + caster_radius -->
+  <xacro:property name="caster_z"
+                  value="${-base_height*0.5 - caster_ground_clearance + caster_radius}"/>
+  <!-- =========================
+       Materials (GLOBAL)
+       ========================= -->
+  <material name="yellow">
     <color rgba="1 1 0 1"/>
   </material>
+  <material name="black">
+    <color rgba="0.05 0.05 0.05 1"/>
+  </material>
+  <!-- Slight transparency to help see the caster under the body in RViz -->
+  <material name="gray">
+    <color rgba="0.6 0.6 0.6 0.7"/>
+  </material>
+  <!-- =========================
+       Links
+       ========================= -->
   <!-- Base Link -->
   <link name="base_link">
     <visual>
+      <origin xyz="0 0 0" rpy="0 0 0"/>
       <geometry>
-        <box size="0.4 0.3 0.1"/>
+        <box size="${base_length} ${base_width} ${base_height}"/>
       </geometry>
+      <material name="gray"/>
     </visual>
     <collision>
+      <origin xyz="0 0 0" rpy="0 0 0"/>
       <geometry>
-        <box size="0.4 0.3 0.1"/>
+        <box size="${base_length} ${base_width} ${base_height}"/>
       </geometry>
     </collision>
     <inertial>
-      <mass value="5.0"/>
-      <origin xyz="0 0 0"/>
-      <inertia ixx="0.1" iyy="0.1" izz="0.1"
+      <origin xyz="0 0 0" rpy="0 0 0"/>
+      <mass value="${base_mass}"/>
+      <!-- Placeholder inertia (OK for now; we can compute later) -->
+      <inertia ixx="0.10" iyy="0.10" izz="0.10"
                ixy="0.0" ixz="0.0" iyz="0.0"/>
     </inertial>
   </link>
-  <!-- Left Wheel -->
+  <!-- Left Drive Wheel -->
   <link name="left_wheel_link">
     <visual>
+      <!-- Cylinder axis is Z by default; rotate so axis aligns with +Y -->
       <origin xyz="0 0 0" rpy="1.5708 0 0"/>
       <geometry>
@@ -44,12 +88,12 @@
     </collision>
     <inertial>
-      <mass value="0.3"/>
       <origin xyz="0 0 0" rpy="0 0 0"/>
-      <!-- conservative inertia guess; we can refine later -->
+      <mass value="${wheel_mass}"/>
+      <!-- Placeholder inertia -->
       <inertia ixx="0.0005" iyy="0.0005" izz="0.0005"
-              ixy="0.0" ixz="0.0" iyz="0.0"/>
+               ixy="0.0" ixz="0.0" iyz="0.0"/>
     </inertial>
   </link>
-  <!-- Right Wheel -->
+  <!-- Right Drive Wheel -->
   <link name="right_wheel_link">
     <visual>
@@ -67,16 +111,39 @@
     </collision>
     <inertial>
-      <mass value="0.3"/>
       <origin xyz="0 0 0" rpy="0 0 0"/>
-      <!-- conservative inertia guess; we can refine later -->
+      <mass value="${wheel_mass}"/>
       <inertia ixx="0.0005" iyy="0.0005" izz="0.0005"
-              ixy="0.0" ixz="0.0" iyz="0.0"/>
+               ixy="0.0" ixz="0.0" iyz="0.0"/>
     </inertial>
   </link>
-  <!-- Joints -->
+  <!-- Passive spherical caster -->
+  <link name="caster_link">
+    <visual>
+      <origin xyz="0 0 0" rpy="0 0 0"/>
+      <geometry>
+        <sphere radius="${caster_radius}"/>
+      </geometry>
+      <material name="black"/>
+    </visual>
+    <collision>
+      <origin xyz="0 0 0" rpy="0 0 0"/>
+      <geometry>
+        <sphere radius="${caster_radius}"/>
+      </geometry>
+    </collision>
+    <inertial>
+      <origin xyz="0 0 0" rpy="0 0 0"/>
+      <mass value="${caster_mass}"/>
+      <inertia ixx="0.0001" iyy="0.0001" izz="0.0001"
+               ixy="0.0" ixz="0.0" iyz="0.0"/>
+    </inertial>
+  </link>
+  <!-- =========================
+       Joints
+       ========================= -->
   <joint name="left_wheel_joint" type="continuous">
     <parent link="base_link"/>
     <child link="left_wheel_link"/>
-    <origin xyz="0 ${wheel_separation * 0.5 + wheel_width*0.5} -${wheel_radius * 0.5}"/>
+    <origin xyz="${drive_wheel_x} ${wheel_separation*0.5} ${drive_wheel_z}" rpy="0 0 0"/>
     <axis xyz="0 1 0"/>
   </joint>
@@ -84,8 +151,15 @@
     <parent link="base_link"/>
     <child link="right_wheel_link"/>
-    <origin xyz="0 -${wheel_separation * 0.5 + wheel_width*0.5} -${wheel_radius * 0.5}"/>
+    <origin xyz="${drive_wheel_x} -${wheel_separation*0.5} ${drive_wheel_z}" rpy="0 0 0"/>
     <axis xyz="0 1 0"/>
   </joint>
-  <!-- Gazebo Harmonic: Thin actuator I/O for wheel joints -->
+  <joint name="caster_joint" type="fixed">
+    <parent link="base_link"/>
+    <child link="caster_link"/>
+    <origin xyz="${caster_x} 0 ${caster_z}" rpy="0 0 0"/>
+  </joint>
+  <!-- =========================
+       Gazebo Harmonic: Thin actuator I/O for drive wheel joints only
+       ========================= -->
   <gazebo>
     <plugin filename="gz-sim-joint-controller-system"
